Commit message: debugging

File: resource/2DrobotArm/robot_3D.urdf (robot description, URDF)
Before this commit: robot 2DrobotArm, 5 links, 4 joints
Joints:
- removed joint link1Tolink3
- added joint link2Tolink3: type revolute, parent link2, child link3, origin xyz=0 0 0.3, axis 1 0 0

File: resource/anymal_c/urdf/anymal.urdf (robot description, URDF)
Before this commit: robot anymal, 78 links, 77 joints
Joints:
- joint LF_HFE: type revolute -> prismatic

Commit message: added debug.cpp

File: resource/2DrobotArm/robot_3D.urdf (robot description, URDF)
Before this commit: robot 2DrobotArm, 5 links, 4 joints
Links:
- link link2: geometry visual cylinder length=0.2 radius=0.02
- link link3: geometry visual cylinder length=0.2 radius=0.02
- link link4: geometry visual cylinder length=0.2 radius=0.02

Commit message: changed 2DrobotArm urdf

File: resource/2DrobotArm/robot_3D.urdf (robot description, URDF)
Before this commit: robot 2DrobotArm, 5 links, 4 joints
Links:
- added link link5, mass 1
- link link4: geometry 
Joints:
- added joint link3Tolink5: type prismatic, parent link3, child link5, origin xyz=0 0 0.3, axis 0 1 0
- joint link3Tolink4: type prismatic -> revolute
